File: clock_board/_saved_cb2.sch (KiCad schematic (older format))
At the start: 39 parts, among them IC1 ATMEGA328-P, P1 POWER, P2 PROGRAMMER, P3 BATT_CONN, P4 LEDB_POWER, P5 LCD_CLK_CONN, P6 DIGIT_POWER, Q1 DGT1, Q2 DGT2, Q3 DGT3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

Commit message: Removed clock reset button.  Improved PCB layout.
Parts:
- C7: footprint Capacitors_Elko_ThroughHole:Elko_vert_20x10mm_RM2.5 -> Capacitors_Elko_ThroughHole:Elko_vert_11.2x6.3mm_RM2.5
Changed lines of the file:
@@
 F 0 "C7" H 9675 1025 50  0000 L CNN
 F 1 "10uF" H 9350 925 50  0000 L CNN
-F 2 "Capacitors_Elko_ThroughHole:Elko_vert_20x10mm_RM2.5" H 9688 775 30  0001 C CNN
+F 2 "Capacitors_Elko_ThroughHole:Elko_vert_11.2x6.3mm_RM2.5" H 9688 775 30  0001 C CNN
 F 3 "" H 9650 925 60  0000 C CNN
 	1    9650 925

Commit message: Updated footprints for DS3231, 4.7k resistors, and battery connection.
Parts:
- R3, R4: footprint Resistors_ThroughHole:Resistor_Horizontal_RM10mm -> Resistors_ThroughHole:Resistor_Horizontal_RM15mm
Changed lines of the file:
@@
 F 0 "R4" V 5155 3075 50  0000 C CNN
 F 1 "4.7k" V 5075 3075 50  0000 C CNN
-F 2 "Resistors_ThroughHole:Resistor_Horizontal_RM10mm" V 5005 3075 30  0001 C CNN
+F 2 "Resistors_ThroughHole:Resistor_Horizontal_RM15mm" V 5005 3075 30  0001 C CNN
 F 3 "" H 5075 3075 30  0000 C CNN
 	1    5075 3075
@@
 F 0 "R3" V 5155 2925 50  0000 C CNN
 F 1 "4.7k" V 5075 2925 50  0000 C CNN
-F 2 "Resistors_ThroughHole:Resistor_Horizontal_RM10mm" V 5005 2925 30  0001 C CNN
+F 2 "Resistors_ThroughHole:Resistor_Horizontal_RM15mm" V 5005 2925 30  0001 C CNN
 F 3 "" H 5075 2925 30  0000 C CNN
 	1    5075 2925
